Commit message: Update ur10e_rg2_hex.urdf

File: description/ur10e_rg2_hex.urdf (robot description, URDF)
Before this commit: robot ur10e_robot_rg2, 19 links, 18 joints
Links:
- link base_link_inertia: geometry collision mesh filename=package://meshes/ur10e/collision/base.stl; visual mesh filename=package://meshes/ur10e/visual/base.dae
- link forearm_link: geometry collision mesh filename=package://meshes/ur10e/collision/forearm.stl; visual mesh filename=package://meshes/ur10e/visual/forearm.dae
- link hex_backplate_link: geometry collision mesh filename=package://meshes/hex/HEX-E_H_QC_v3_backplate_A.stl scale=0.001 0.001 0.001; visual mesh filename=package://meshes/hex/HEX-E_H_QC_v3_backplate_A.stl scale=0.001 0.001 0.001
- link hex_link: geometry collision mesh filename=package://meshes/hex/HEX_QC_2.STL scale=0.001 0.001 0.001; visual mesh filename=package://meshes/hex/HEX_QC_2.STL scale=0.001 0.001 0.001
- link left_inner_finger: geometry collision mesh filename=package://meshes/onrobot_rg2/collision/inner_finger.stl; visual mesh filename=package://meshes/onrobot_rg2/visual/inner_finger.stl
- link left_inner_knuckle: geometry collision mesh filename=package://meshes/onrobot_rg2/collision/inner_knuckle.stl; visual mesh filename=package://meshes/onrobot_rg2/visual/inner_knuckle.stl
- link left_outer_knuckle: geometry collision mesh filename=package://meshes/onrobot_rg2/collision/outer_knuckle.stl; visual mesh filename=package://meshes/onrobot_rg2/visual/outer_knuckle.stl
- link onrobot_rg2_base_link: geometry collision mesh filename=package://meshes/onrobot_rg2/collision/base_link.stl; visual mesh filename=package://meshes/onrobot_rg2/visual/base_link.stl
- link right_inner_finger: geometry collision mesh filename=package://meshes/onrobot_rg2/collision/inner_finger.stl; visual mesh filename=package://meshes/onrobot_rg2/visual/inner_finger.stl
- link right_inner_knuckle: geometry collision mesh filename=package://meshes/onrobot_rg2/collision/inner_knuckle.stl; visual mesh filename=package://meshes/onrobot_rg2/visual/inner_knuckle.stl
- link right_outer_knuckle: geometry collision mesh filename=package://meshes/onrobot_rg2/collision/outer_knuckle.stl; visual mesh filename=package://meshes/onrobot_rg2/visual/outer_knuckle.stl
- link shoulder_link: geometry collision mesh filename=package://meshes/ur10e/collision/shoulder.stl; visual mesh filename=package://meshes/ur10e/visual/shoulder.dae
- link upper_arm_link: geometry collision mesh filename=package://meshes/ur10e/collision/upperarm.stl; visual mesh filename=package://meshes/ur10e/visual/upperarm.dae
- link wrist_1_link: geometry collision mesh filename=package://meshes/ur10e/collision/wrist1.stl; visual mesh filename=package://meshes/ur10e/visual/wrist1.dae
- link wrist_2_link: geometry collision mesh filename=package://meshes/ur10e/collision/wrist2.stl; visual mesh filename=package://meshes/ur10e/visual/wrist2.dae
- link wrist_3_link: geometry collision mesh filename=package://meshes/ur10e/collision/wrist3.stl; visual mesh filename=package://meshes/ur10e/visual/wrist3.dae

Commit message: change the UR10e description file

File: description/ur10e_rg2_hex.urdf (robot description, URDF)
Before this commit: robot ur10e_robot_rg2, 19 links, 18 joints
Joints:
- joint wrist_3_hand: origin xyz=0 0 0.05 rpy=3.14159265359 3.14159265359 -3.14159265359 -> xyz=0 0 0.05 rpy=3.14159265359 3.14159265359 1.57079632679
- joint wrist_3_hex_backplate: origin xyz=0 0 0 rpy=-1.57079632659 3.14159265359 3.14159265359 -> xyz=0 0 0 rpy=-1.57079632659 3.14159265359 0
